File: hardware/General-Purpose-SMD/General-Purpose-SMD.kicad_pcb (KiCad board)
At the start: 2 copper layers, 56 x 15 mm, 9 parts, among them J1 Screw_Terminal_01x03, J4 Screw_Terminal_01x03, J5 Screw_Terminal_01x03, K1 G6K-2F-Y-TR DC12, K2 G6K-2F-Y-TR DC12

Commit message: added picture
Parts:
- removed the REF** at (120.4, 63.6)
- added D1: LED, LED_SMD:LED_0805_2012Metric_Pad1.15x1.40mm_HandSolder, F.Cu at (134.4, 57.1)
- added D2: LED, LED_SMD:LED_0805_2012Metric_Pad1.15x1.40mm_HandSolder, F.Cu at (134.4, 69.6)
- added R3: 4k7, custom_kicad_lib_sk:R_0603_smalltext, F.Cu at (130.2, 57.0)
- added R4: 4k7, custom_kicad_lib_sk:R_0603_smalltext, F.Cu at (130.2, 69.8)
Routing:
- net /relay1/V+: track 9.22 -> 70.9 mm
- net /relay1/Coil1: track 15.7 -> 31.7 mm
- net /relay1/Coil2: track 20.2 -> 32.6 mm
- net Net-(D2-A): track 0.00 -> 2.36 mm
- net Net-(D1-A): track 0.00 -> 2.31 mm
- net /relay1/NC1: track 36.1 -> 35.6 mm
- net /relay1/NO2: track 44.1 -> 44.4 mm, vias 3 -> 5
