File: hardware/General-Purpose-SMD/relay.kicad_sch (KiCad schematic)
At the start: 7 parts, among them J1 Screw_Terminal_01x03, J4 Screw_Terminal_01x03, J5 Screw_Terminal_01x03, K1 G6K-2F-Y-TR DC12, K2 G6K-2F-Y-TR DC12

Commit message: added picture
Parts:
- added D1, D2: LED, LED_SMD:LED_0805_2012Metric_Pad1.15x1.40mm_HandSolder, symbol custom_kicad_lib_sk:LED
- added R3, R4: 4k7, custom_kicad_lib_sk:R_0603_smalltext, symbol resistors_0603:R_4k7_0603
Connections:
- net Coil1: now also D1.1 (K)
- net Coil2: now also D2.1 (K)
- net V+: now also R3.1, R4.1
- new net: D2.2 (A), R4.2
- new net: D1.2 (A), R3.2
